File: pcb/mriya-left/mriya-left.kicad_pcb (KiCad board)
At the start: 2 copper layers, 137 x 84 mm, 59 parts, among them J1 PJ-320A, J2 Battery, J3 nice!view, SW1 SW_PUSH, SW10 SW_PUSH, SW11 SW_PUSH, SW12 SW_PUSH, SW13 SW_PUSH, SW14 SW_PUSH, SW15 SW_PUSH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

Commit message: updated references
Parts:
- renumbered J3 to J1, J1 to J3, SW22 to PSW1

Commit message: updated references
Parts:
- renumbered J2 to J5
