File: pcb/mriya-left/mriya-left.kicad_sch (KiCad schematic)
At the start: 55 parts, among them J1 PJ-320A, J2 Battery, J3 nice!view, SW1 SW_PUSH, SW10 SW_PUSH, SW11 SW_PUSH, SW12 SW_PUSH, SW13 SW_PUSH, SW14 SW_PUSH, SW15 SW_PUSH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

Commit message: updated references
Parts:
- U1: footprint mriya:ProMicro_v3 -> mriya:ProMicro
- renumbered J3 to J1, J1 to J3, SW22 to PSW1
Changed lines of the file:
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@@
       (effects (font (size 1.524 1.524)))
     )
-    (property "Footprint" "mriya:ProMicro_v3" (at 49.53 71.12 0)
+    (property "Footprint" "mriya:ProMicro" (at 49.53 71.12 0)
       (effects (font (size 1.524 1.524)) hide)
     )
@@
   (symbol (lib_id "Switch:SW_SPDT") (at 111.0742 34.29 0) (unit 1)
     (in_bom yes) (on_board yes) (dnp no)
-    (property "Reference" "SW22" (at 111.0742 27.051 0)
+    (property "Reference" "PSW1" (at 111.0742 27.051 0)
       (effects (font (size 1.27 1.27)))
     )
@@
       (project "mriya-left"
         (path "/eb62da78-dfd8-4bde-9993-50d36b1638e4"
-          (reference "SW22") (unit 1)
+          (reference "PSW1") (unit 1)
         )
       )
@@
   (symbol (lib_id "corne-cherry-left-rescue:MJ-4PP-9-kbd") (at 39.37 103.505 0) (unit 1)
     (in_bom yes) (on_board yes) (dnp no)
-    (property "Reference" "J1" (at 39.37 99.695 0)
+    (property "Reference" "J3" (at 39.37 99.695 0)
       (effects (font (size 1.27 1.27)))
     )
@@
       (project "mriya-left"
         (path "/eb62da78-dfd8-4bde-9993-50d36b1638e4"
-          (reference "J1") (unit 1)
+          (reference "J3") (unit 1)
         )
       )
@@
   (symbol (lib_id "Connector_Generic:Conn_01x05") (at 40.64 80.645 180) (unit 1)
     (in_bom yes) (on_board yes) (dnp no)
-    (property "Reference" "J3" (at 40.64 71.755 0)
+    (property "Reference" "J1" (at 40.64 71.755 0)
       (effects (font (size 1.27 1.27)))
     )
@@
       (project "mriya-left"
         (path "/eb62da78-dfd8-4bde-9993-50d36b1638e4"
-          (reference "J3") (unit 1)
-        )
-      )
+          (reference "J1") (unit 1)
+        )
+      )

Commit message: updated references
Parts:
- renumbered J2 to J5
Changed lines of the file:
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@@
   (symbol (lib_id "Connector:Conn_01x02_Female") (at 128.27 34.29 0) (unit 1)
     (in_bom yes) (on_board yes) (dnp no)
-    (property "Reference" "J2" (at 128.9812 34.8996 0)
+    (property "Reference" "J5" (at 128.9812 34.8996 0)
       (effects (font (size 1.27 1.27)) (justify left))
     )
@@
       (project "mriya-left"
         (path "/eb62da78-dfd8-4bde-9993-50d36b1638e4"
-          (reference "J2") (unit 1)
+          (reference "J5") (unit 1)
         )
       )
