File: pcb/mriya-right/mriya-right.kicad_pcb (KiCad board)
At the start: 2 copper layers, 137 x 84 mm, 59 parts, among them J4 PJ-320A, J5 Battery, J6 nice!view, SW22 SW_PUSH, SW23 SW_PUSH, SW24 SW_PUSH, SW25 SW_PUSH, SW26 SW_PUSH, SW27 SW_PUSH, SW28 SW_PUSH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

Commit message: updated references
Parts:
- renumbered J6 to J2, SW44 to PSW2, RSW3 to RSW2

Commit message: updated references
Parts:
- renumbered J5 to J6
