File: pcb/mriya-right/mriya-right.kicad_sch (KiCad schematic)
At the start: 55 parts, among them J4 PJ-320A, J5 Battery, J6 nice!view, SW22 SW_PUSH, SW23 SW_PUSH, SW24 SW_PUSH, SW25 SW_PUSH, SW26 SW_PUSH, SW27 SW_PUSH, SW28 SW_PUSH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

Commit message: updated references
Parts:
- renumbered J6 to J2, SW44 to PSW2, RSW3 to RSW2
Other:
- moved on the sheet: RSW2
Changed lines of the file:
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@@
     )
   )
-  (global_label "reset_r" (shape input) (at 83.82 101.6 180) (fields_autoplaced)
+  (global_label "reset_r" (shape input) (at 111.76 100.33 180) (fields_autoplaced)
     (effects (font (size 1.524 1.524)) (justify right))
-    (property "Intersheetrefs" "${INTERSHEET_REFS}" (at -154.305 2.54 0)
+    (property "Intersheetrefs" "${INTERSHEET_REFS}" (at -126.365 1.27 0)
       (effects (font (size 1.27 1.27)) hide)
     )
@@
   (symbol (lib_id "Connector_Generic:Conn_01x05") (at 41.91 74.3204 180) (unit 1)
     (in_bom yes) (on_board yes) (dnp no)
-    (property "Reference" "J6" (at 41.91 65.4304 0)
+    (property "Reference" "J2" (at 41.91 65.4304 0)
       (effects (font (size 1.27 1.27)))
     )
@@
       (project "mriya-right"
         (path "/e02cb072-403e-4f41-9df6-6bdac0d01d9b"
-          (reference "J6") (unit 1)
+          (reference "J2") (unit 1)
         )
       )
@@
     )
   )
-  (symbol (lib_id "corne-cherry-right-rescue:SW_PUSH-kbd") (at 91.44 101.6 0) (unit 1)
-    (in_bom yes) (on_board yes) (dnp no)
-    (property "Reference" "RSW3" (at 95.25 98.806 0)
-      (effects (font (size 1.27 1.27)))
-    )
-    (property "Value" "SW_PUSH" (at 91.44 103.632 0)
-      (effects (font (size 1.27 1.27)))
-    )
-    (property "Footprint" "mriya:RSW_4.5x4.5_vert" (at 91.44 101.6 0)
-      (effects (font (size 1.27 1.27)) hide)
-    )
-    (property "Datasheet" "" (at 91.44 101.6 0)
-      (effects (font (size 1.27 1.27)))
-    )
-    (pin "1")
-    (pin "2")
-    (instances
-      (project "mriya-right"
-        (path "/e02cb072-403e-4f41-9df6-6bdac0d01d9b"
-          (reference "RSW3") (unit 1)
+  (symbol (lib_id "corne-cherry-right-rescue:SW_PUSH-kbd") (at 119.38 100.33 0) (unit 1)
+    (in_bom yes) (on_board yes) (dnp no)
+    (property "Reference" "RSW2" (at 123.19 97.536 0)
+      (effects (font (size 1.27 1.27)))
+    )
+    (property "Value" "SW_PUSH" (at 119.38 102.362 0)
+      (effects (font (size 1.27 1.27)))
+    )
+    (property "Footprint" "mriya:RSW_4.5x4.5_vert" (at 119.38 100.33 0)
+      (effects (font (size 1.27 1.27)) hide)
+    )
+    (property "Datasheet" "" (at 119.38 100.33 0)
+      (effects (font (size 1.27 1.27)))
+    )
+    (pin "1")
+    (pin "2")
+    (instances
+      (project "mriya-right"
+        (path "/e02cb072-403e-4f41-9df6-6bdac0d01d9b"
+          (reference "RSW2") (unit 1)
         )
       )
@@
   (symbol (lib_id "Switch:SW_SPDT") (at 114.3 31.75 0) (unit 1)
     (in_bom yes) (on_board yes) (dnp no)
-    (property "Reference" "SW44" (at 110.7694 24.638 0)
+    (property "Reference" "PSW2" (at 110.7694 24.638 0)
       (effects (font (size 1.27 1.27)))
     )
@@
       (project "mriya-right"
         (path "/e02cb072-403e-4f41-9df6-6bdac0d01d9b"
-          (reference "SW44") (unit 1)
+          (reference "PSW2") (unit 1)
         )
       )
@@
     )
   )
-  (symbol (lib_id "power:GNDA") (at 99.06 101.6 0) (unit 1)
-    (in_bom yes) (on_board yes) (dnp no)
-    (property "Reference" "#PWR0108" (at 99.06 107.95 0)
-      (effects (font (size 1.27 1.27)) hide)
-    )
-    (property "Value" "GNDA" (at 99.06 105.41 0)
-      (effects (font (size 1.27 1.27)))
-    )
-    (property "Footprint" "" (at 99.06 101.6 0)
-      (effects (font (size 1.27 1.27)) hide)
-    )
-    (property "Datasheet" "" (at 99.06 101.6 0)
-      (effects (font (size 1.27 1.27)) hide)
-    )
+  (symbol (lib_id "power:GNDA") (at 127 100.33 0) (unit 1)
+    (in_bom yes) (on_board yes) (dnp no)
+    (property "Reference" "#PWR0108" (at 127 106.68 0)
+      (effects (font (size 1.27 1.27)) hide)
+    )
+    (property "Value" "GNDA" (at 127 104.14 0)
+      (effects (font (size 1.27 1.27)))
+    )
+    (property "Footprint" "" (at 127 100.33 0)
+      (effects (font (size 1.27 1.27)) hide)
+    )
+    (property "Datasheet" "" (at 127 100.33 0)
+      (effects (font (size 1.27 1.27)) hide)
+    )

Commit message: updated references
Parts:
- renumbered J5 to J6
Changed lines of the file:
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@@
   (symbol (lib_id "Connector:Conn_01x02_Female") (at 129.54 26.67 0) (unit 1)
     (in_bom yes) (on_board yes) (dnp no)
-    (property "Reference" "J5" (at 130.2512 27.2796 0)
+    (property "Reference" "J6" (at 130.2512 27.2796 0)
       (effects (font (size 1.27 1.27)) (justify left))
     )
@@
       (project "mriya-right"
         (path "/e02cb072-403e-4f41-9df6-6bdac0d01d9b"
-          (reference "J5") (unit 1)
+          (reference "J6") (unit 1)
         )
       )
